File: eagle_files/main.sch (EAGLE design)
At the start: 9 parts, among them X1 22-23-2021

Commit message: fix board design
Parts:
- removed Q1: (no value), crystal:CRYSTALTC26H
- removed TP1, TP2: TPTP12R, testpad:TPTP12R
Connections:
- removed net N$14: TP1.TP
- net GND: no longer TP2.TP
- net N$10: no longer Q1.1
- net N$12: no longer Q1.2
Changed lines of the file:
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@@
 <part name="GND6" library="supply1" deviceset="GND" device=""/>
 <part name="+3V6" library="supply1" deviceset="+3V3" device=""/>
-<part name="Q1" library="crystal" deviceset="CRYSTAL" device="TC26H"/>
-<part name="TP1" library="testpad" deviceset="TP" device="TP12R"/>
-<part name="TP2" library="testpad" deviceset="TP" device="TP12R"/>
-<part name="GND7" library="supply1" deviceset="GND" device=""/>
 </parts>
 <sheets>
@@
 <text x="-2.54" y="17.78" size="1.778" layer="91" rot="R90">MISO</text>
 <text x="12.7" y="17.78" size="1.778" layer="91" rot="R90">CS</text>
+<rectangle x1="78.74" y1="68.58" x2="81.28" y2="71.12" layer="91" rot="R180"/>
+<rectangle x1="78.74" y1="63.5" x2="81.28" y2="66.04" layer="91" rot="R180"/>
+<rectangle x1="-35.56" y1="63.5" x2="-33.02" y2="66.04" layer="91"/>
 </plain>
 <instances>
@@
 <instance part="GND6" gate="1" x="20.32" y="78.74" rot="R90"/>
 <instance part="+3V6" gate="G$1" x="15.24" y="83.82"/>
-<instance part="Q1" gate="G$1" x="81.28" y="66.04" rot="R90"/>
-<instance part="TP1" gate="G$1" x="-35.56" y="66.04"/>
-<instance part="TP2" gate="G$1" x="-38.1" y="66.04"/>
-<instance part="GND7" gate="1" x="-38.1" y="60.96"/>
 </instances>
 <busses>
@@
 <wire x1="17.78" y1="78.74" x2="20.32" y2="78.74" width="0.1524" layer="91"/>
 <junction x="17.78" y="78.74"/>
-</segment>
-<segment>
-<pinref part="TP2" gate="G$1" pin="TP"/>
-<pinref part="GND7" gate="1" pin="GND"/>
 </segment>
 </net>
@@
 </segment>
 </net>
-<net name="N$12" class="0">
-<segment>
-<pinref part="U$1" gate="G$1" pin="18"/>
-<pinref part="Q1" gate="G$1" pin="2"/>
-<wire x1="66.04" y1="68.58" x2="81.28" y2="68.58" width="0.1524" layer="91"/>
-</segment>
-</net>
 <net name="N$10" class="0">
 <segment>
-<pinref part="Q1" gate="G$1" pin="1"/>
-<wire x1="76.2" y1="63.5" x2="81.28" y2="63.5" width="0.1524" layer="91"/>
 <pinref part="U$1" gate="G$1" pin="19"/>
-<wire x1="66.04" y1="71.12" x2="76.2" y2="71.12" width="0.1524" layer="91"/>
-<wire x1="76.2" y1="71.12" x2="76.2" y2="63.5" width="0.1524" layer="91"/>
+<wire x1="66.04" y1="71.12" x2="78.74" y2="71.12" width="0.1524" layer="91"/>
 </segment>
 </net>
@@
 <wire x1="-5.08" y1="66.04" x2="20.32" y2="66.04" width="0.1524" layer="91"/>
 <wire x1="-5.08" y1="68.58" x2="-5.08" y2="66.04" width="0.1524" layer="91"/>
-<pinref part="TP1" gate="G$1" pin="TP"/>
-</segment>
-</net>
+</segment>
+</net>
+<net name="N$12" class="0">
+<segment>
+<pinref part="U$1" gate="G$1" pin="18"/>
+<wire x1="66.04" y1="68.58" x2="73.66" y2="68.58" width="0.1524" layer="91"/>
+<wire x1="73.66" y1="68.58" x2="73.66" y2="60.96" width="0.1524" layer="91"/>
+<wire x1="73.66" y1="60.96" x2="78.74" y2="60.96" width="0.1524" layer="91"/>
+<wire x1="78.74" y1="66.04" x2="78.74" y2="60.96" width="0.1524" layer="91"/>
+</segment>
+</net>
